Commit message: update cutter/env models with simpler models

File: models/trellis-model.urdf (robot description, URDF)
Before this commit: robot test_tree, 1 links, 0 joints
Links:
- link baseLink: mass .0 -> 10.0; geometry collision mesh filename=trellis-model-rect.obj scale=1 1 1; visual mesh filename=trellis-model-rect.obj scale=1 1 1

Commit message: creation of basic gym environment

File: models/trellis-model.urdf (robot description, URDF)
Before this commit: robot test_tree, 1 links, 0 joints
Links:
- added link target_1; visual sphere center=0.0 0.0 0.0 radius=0.005
- added link target_2; visual sphere center=0.0 0.0 0.0 radius=0.005
Joints:
- added joint world_target_1: type fixed, parent baseLink, child target_1, origin xyz=0.0 0.2 0.8 rpy=0 0 0
- added joint world_target_2: type fixed, parent baseLink, child target_2, origin xyz=0.0 -0.2 0.8 rpy=0 0 0

Commit message: basic learning demonstration running

File: models/trellis-model.urdf (robot description, URDF)
Before this commit: robot test_tree, 3 links, 2 joints
Links:
- link target_1: geometry collision cylinder length=0.12 radius=0.0025; visual cylinder length=0.12 radius=0.0025
- link target_2: geometry collision cylinder length=0.12 radius=0.0025; visual cylinder length=0.12 radius=0.0025
Joints:
- joint world_target_2: origin xyz=0.0 -0.2 0.8 rpy=0 0 0 -> xyz=0.0 -0.2 0.75 rpy=0 0 0
