Commit message: modifications for cross-platform compatibility

File: robots/ur5e_cutter_new_calibrated_precise.urdf (robot description, URDF)
Before this commit: robot ur5e, 17 links, 16 joints
Links:
- link base_link: geometry collision mesh filename=ur5e/collision/base.stl; visual mesh filename=ur5e/visual/base.dae
- link camera_mount: geometry collision box size=0.121 0.060 0.050; visual mesh filename=ur5e/visual/camera_mount.dae scale=1.0 1.0 1.0
- link cutter: geometry collision box size=0.02 0.05 0.08; collision box size=0.07 0.084 0.06
- link forearm_link: geometry collision mesh filename=ur5e/collision/forearm.stl; visual mesh filename=ur5e/visual/forearm.dae
- link shoulder_link: geometry collision mesh filename=ur5e/collision/shoulder.stl; visual mesh filename=ur5e/visual/shoulder.dae
- link upper_arm_link: geometry collision mesh filename=ur5e/collision/upperarm.stl; visual mesh filename=ur5e/visual/upperarm.dae
- link wrist_1_link: geometry collision mesh filename=ur5e/collision/wrist1.stl; visual mesh filename=ur5e/visual/wrist1.dae
- link wrist_2_link: geometry collision mesh filename=ur5e/collision/wrist2.stl; visual mesh filename=ur5e/visual/wrist2.dae
- link wrist_3_link: geometry collision mesh filename=ur5e/collision/wrist3.stl; visual mesh filename=ur5e/visual/wrist3.dae

Commit message: UR model updates, state resetting for servoing

File: robots/ur5e_cutter_new_calibrated_precise.urdf (robot description, URDF)
Before this commit: robot ur5e, 17 links, 16 joints
Links:
- link cutter: geometry collision mesh filename=ur5e/collision/new_cutter.stl scale=1.0 1.0 1.0; visual mesh filename=ur5e/visual/new_cutter.dae scale=1.0 1.0 1.0
- link mount: geometry collision box size=0.5 0.5 0.75711; visual mesh filename=ur5e/visual/robot_cart.obj
Joints:
- joint mount_base_joint: origin xyz=0.0 0.0 0.75 rpy=0.0 0.0 0.0 -> xyz=0.0 0.0 0.0 rpy=0.0 0.0 -1.5708
- joint world_joint: origin xyz=0.0 0.0 0.0 rpy=0.0 0.0 0.0 -> xyz=0.0 0.0 0.75711 rpy=0.0 0.0 1.5708

Commit message: update cutter/env models with simpler models

File: robots/ur5e_cutter_new_calibrated_precise.urdf (robot description, URDF)
Before this commit: robot ur5e, 17 links, 16 joints
Links:
- link cutter: geometry collision mesh filename=ur5e/collision/new_cutter_decimated.stl scale=1.0 1.0 1.0; visual mesh filename=ur5e/visual/new_cutter.dae scale=1.0 1.0 1.0

Commit message: convexified cutter model for collision detection

File: robots/ur5e_cutter_new_calibrated_precise.urdf (robot description, URDF)
Before this commit: robot ur5e, 17 links, 16 joints
Links:
- link cutter: geometry collision mesh filename=ur5e/collision/new-cutter-convexified.obj scale=1.0 1.0 1.0; visual mesh filename=ur5e/collision/new-cutter-convexified.obj scale=1.0 1.0 1.0

Commit message: code automatically points camera towards cutpoint, fixes error with TINY_RENDERER failing when coincident with joint

File: robots/ur5e_cutter_new_calibrated_precise.urdf (robot description, URDF)
Before this commit: robot ur5e, 17 links, 16 joints
Links:
- removed link camera_mount
Joints:
- removed joint camera_mount
- joint cutter: parent camera_mount -> tool0

Commit message: Updated cutter mesh to have proper wood texturing

File: robots/ur5e_cutter_new_calibrated_precise.urdf (robot description, URDF)
Before this commit: robot ur5e, 16 links, 15 joints
Links:
- link cutpoint: geometry visual sphere radius=0.00001
- link cutter: geometry collision mesh filename=ur5e/collision/new-cutter-convexified.obj scale=1.0 1.0 1.0; visual mesh filename=ur5e/visual/cutter_wooden.obj scale=1.0 1.0 1.0
- link endpoint: geometry visual sphere radius=0.00001

Commit message: cutter model update

File: robots/ur5e_cutter_new_calibrated_precise.urdf (robot description, URDF)
Before this commit: robot ur5e, 16 links, 15 joints
Links:
- link cutter: geometry collision mesh filename=ur5e/collision/cutter_wooden_convexified.obj scale=1.0 1.0 1.0; visual mesh filename=ur5e/visual/cutter_wooden.obj scale=1.0 1.0 1.0
Joints:
- joint endpoint: origin xyz=-0.09286 -0.00511 0.09707 rpy=0 0 3.14159 -> xyz=-0.09425 -0.00511 0.09707 rpy=0 0 3.14159
