Commit message: final mount model, added cropping and downsampling, enlarged mouth collision to account for physics

File: robots/ur5e_cutter_new_calibrated_precise_level.urdf (robot description, URDF)
Before this commit: robot ur5e, 16 links, 15 joints
Links:
- link cutter: geometry collision mesh filename=ur5e/collision/cutter_top_mount.obj scale=1.0 1.0 1.0; visual mesh filename=ur5e/visual/cutter_top_mount.obj scale=1.0 1.0 1.0
Joints:
- joint endpoint: origin xyz=-0.063175 0 0.20364 rpy=0 0 0 -> xyz=-0.063175 0 0.12864 rpy=0 0 0
